File: Heat_Ctrl.sch (KiCad schematic (older format))
At the start: 35 parts, among them K1 SRD-05VDC-SL-C, K2 SRD-05VDC-SL-C, P1 PWR, P2 DISPLAY, P3 IR_REC, P4 IIC_EXT, P5 Mains, P6 Touch, P7 TH1, P8 TH2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

Commit message: IR Update
Parts:
- added C7: 1u, Capacitors_SMD:C_0805, symbol C_Small
- added R10: 180, Resistors_SMD:R_0805, symbol R_Small
- added R9: 10K, Resistors_SMD:R_0805, symbol R_Small
Connections:
- wire segments 160 -> 168
Changed lines of the file:
@@
 LIBS:contrib
 LIBS:valves
-LIBS:bluepill_breakouts
 LIBS:heat_ctrl
 LIBS:Heat_Ctrl-cache
@@
 L GND #PWR023
 U 1 1 5A1A560E
-P 3600 2250
-F 0 "#PWR023" H 3600 2000 50  0001 C CNN
-F 1 "GND" H 3600 2100 50  0000 C CNN
-F 2 "" H 3600 2250 50  0000 C CNN
-F 3 "" H 3600 2250 50  0000 C CNN
-	1    3600 2250
-	1    0    0    -1
-$EndComp
-Wire Wire Line
-	3600 2200 3600 2250
+P 3375 2300
+F 0 "#PWR023" H 3375 2050 50  0001 C CNN
+F 1 "GND" H 3375 2150 50  0000 C CNN
+F 2 "" H 3375 2300 50  0000 C CNN
+F 3 "" H 3375 2300 50  0000 C CNN
+	1    3375 2300
+	1    0    0    -1
+$EndComp
+Wire Wire Line
+	3600 2200 3600 2275
 $Comp
 L +3.3V #PWR024
 U 1 1 5A1A579E
-P 3600 2050
-F 0 "#PWR024" H 3600 1900 50  0001 C CNN
-F 1 "+3.3V" H 3600 2190 50  0000 C CNN
-F 2 "" H 3600 2050 50  0000 C CNN
-F 3 "" H 3600 2050 50  0000 C CNN
-	1    3600 2050
-	1    0    0    -1
-$EndComp
-Wire Wire Line
-	3600 2050 3600 2100
-Wire Wire Line
-	1400 6700 900  6700
+P 3025 1975
+F 0 "#PWR024" H 3025 1825 50  0001 C CNN
+F 1 "+3.3V" H 3025 2115 50  0000 C CNN
+F 2 "" H 3025 1975 50  0000 C CNN
+F 3 "" H 3025 1975 50  0000 C CNN
+	1    3025 1975
+	1    0    0    -1
+$EndComp
+Wire Wire Line
+	3600 2025 3600 2100
+Wire Wire Line
+	700  6700 1400 6700
 Text Label 900  6700 0    60   ~ 0
 IR_IN
@@
 	1    0    0    -1
 $EndComp
+$Comp
+L R_Small R9
+U 1 1 5A2030B3
+P 700 6550
+F 0 "R9" H 730 6570 50  0000 L CNN
+F 1 "10K" H 730 6510 50  0000 L CNN
+F 2 "Resistors_SMD:R_0805" H 700 6550 50  0001 C CNN
+F 3 "" H 700 6550 50  0000 C CNN
+	1    700  6550
+	1    0    0    -1
+$EndComp
+Wire Wire Line
+	700  6650 700  6700
+$Comp
+L +3.3V #PWR034
+U 1 1 5A203905
+P 700 6400
+F 0 "#PWR034" H 700 6250 50  0001 C CNN
+F 1 "+3.3V" H 700 6540 50  0000 C CNN
+F 2 "" H 700 6400 50  0000 C CNN
+F 3 "" H 700 6400 50  0000 C CNN
+	1    700  6400
+	1    0    0    -1
+$EndComp
+Wire Wire Line
+	700  6400 700  6450
+Wire Wire Line
+	3375 2250 3375 2300
+Wire Wire Line
+	3600 2275 3375 2275
+Connection ~ 3375 2275
+Wire Wire Line
+	3275 2025 3600 2025
+$Comp
+L R_Small R10
+U 1 1 5A20CF3E
+P 3175 2025
+F 0 "R10" H 3205 2045 50  0000 L CNN
+F 1 "180" H 3205 1985 50  0000 L CNN
+F 2 "Resistors_SMD:R_0805" H 3175 2025 50  0001 C CNN
+F 3 "" H 3175 2025 50  0000 C CNN
+	1    3175 2025
+	0    -1   -1   0
+$EndComp
+Wire Wire Line
+	3025 1975 3025 2025
+Wire Wire Line
+	3025 2025 3075 2025
+$Comp
+L C_Small C7
+U 1 1 5A2047C3
+P 3375 2150
+F 0 "C7" H 3385 2220 50  0000 L CNN
+F 1 "1u" H 3385 2070 50  0000 L CNN
+F 2 "Capacitors_SMD:C_0805" H 3375 2150 50  0001 C CNN
+F 3 "" H 3375 2150 50  0000 C CNN
+	1    3375 2150
+	1    0    0    -1
+$EndComp
+Wire Wire Line
+	3375 2050 3375 2025
+Connection ~ 3375 2025
 $EndSCHEMATC
